File: power-bridge/power-bridge.brd (EAGLE design)
At the start: 9.8 x 22.4 mm, 3 parts, among them X2 PCB-03-2

Commit message: Finalize Power slot
Parts:
- X2: value PCB-03-2 -> CON-MA03-2PCB_EDGE; device sanisimov:PCB_EDGE_2X3 -> sanisimov:PCB_EDGE_03-2
Changed lines of the file:
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@@
 <?xml version="1.0" encoding="utf-8"?>
 <!DOCTYPE eagle SYSTEM "eagle.dtd">
-<eagle version="9.4.2">
+<eagle version="9.5.1">
 <drawing>
 <settings>
@@
 </autorouter>
 <elements>
-<element name="X1" library="sanisimov" package="FE05-2" package3d_urn="urn:adsk.eagle:package:8170/1" value="" x="7.62" y="24.99" smashed="yes" rot="R90">
-<attribute name="MF" value="" x="7.62" y="24.99" size="1.778" layer="27" rot="R90" display="off"/>
-<attribute name="MPN" value="" x="7.62" y="24.99" size="1.778" layer="27" rot="R90" display="off"/>
-<attribute name="OC_FARNELL" value="unknown" x="7.62" y="24.99" size="1.778" layer="27" rot="R90" display="off"/>
-<attribute name="OC_NEWARK" value="unknown" x="7.62" y="24.99" size="1.778" layer="27" rot="R90" display="off"/>
-<attribute name="POPULARITY" value="3" x="7.62" y="24.99" size="1.778" layer="27" rot="R90" display="off"/>
+<element name="X1" library="sanisimov" package="FE05-2" value="" x="7.62" y="24.99" smashed="yes" rot="R90">
 <attribute name="VALUE" x="12.319" y="21.815" size="1.27" layer="27" ratio="10" rot="R90"/>
 </element>
-<element name="X2" library="sanisimov" package="PCB_EDGE_2X3" value="PCB-03-2" x="7.62" y="2.54" smashed="yes"/>
-<element name="U$2" library="sanisimov" package="MOUNTINGHOLE_2.7_PLATEDTHIN" value="MOUNTINGHOLE2.7THIN" x="7.62" y="15.04" smashed="yes"/>
+<element name="X2" library="sanisimov" package="PCB_EDGE_03-2" value="CON-MA03-2PCB_EDGE" x="7.62" y="2.54" smashed="yes"/>
+<element name="U$2" library="sanisimov" package="MOUNTINGHOLE_2.7_PLATEDTHIN" value="MOUNTINGHOLE2.7THIN" x="7.62" y="15.04" smashed="yes">
+<attribute name="BOM" value="EXCLUDE" x="7.62" y="15.04" size="1.778" layer="27" display="off"/>
+</element>
 </elements>
 <signals>
@@
 </board>
 </drawing>
-<compatibility>
-<note version="8.3" severity="warning">
-Since Version 8.3, EAGLE supports URNs for individual library
-assets (packages, symbols, and devices). The URNs of those assets
-will not be understood (or retained) with this version.
-</note>
-<note version="8.3" severity="warning">
-Since Version 8.3, EAGLE supports the association of 3D packages
-with devices in libraries, schematics, and board files. Those 3D
-packages will not be understood (or retained) with this version.
-</note>
-</compatibility>
 </eagle>
