File: power-bridge/power-bridge.sch (EAGLE design)
At the start: 3 parts, among them X2 PCB-03-2

Commit message: Finalize Power slot
Parts:
- X1: device sanisimov:FE05-2 -> sanisimov:CON-FE05-2
- X2: value PCB-03-2 -> CON-MA03-2PCB_EDGE; device sanisimov:PCB-03-2 -> sanisimov:CON-MA03-2PCB_EDGE
Changed lines of the file:
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@@
 <?xml version="1.0" encoding="utf-8"?>
 <!DOCTYPE eagle SYSTEM "eagle.dtd">
-<eagle version="9.4.2">
+<eagle version="9.5.1">
 <drawing>
 <settings>
-<setting alwaysvectorfont="yes"/>
+<setting alwaysvectorfont="no"/>
 <setting verticaltext="up"/>
 </settings>
@@
 </classes>
 <parts>
-<part name="X1" library="sanisimov" deviceset="FE05-2" device="" package3d_urn="urn:adsk.eagle:package:8170/1"/>
+<part name="X1" library="sanisimov" deviceset="CON-FE05-2" device=""/>
 <part name="U$1" library="sanisimov" deviceset="GND" device=""/>
-<part name="X2" library="sanisimov" deviceset="PCB-03-2" device=""/>
+<part name="X2" library="sanisimov" deviceset="CON-MA03-2" device="PCB_EDGE"/>
 <part name="U$2" library="sanisimov" deviceset="MOUNTINGHOLE" device="2.7THIN" value="MOUNTINGHOLE2.7THIN"/>
 </parts>
@@
 </schematic>
 </drawing>
-<compatibility>
-<note version="8.3" severity="warning">
-Since Version 8.3, EAGLE supports URNs for individual library
-assets (packages, symbols, and devices). The URNs of those assets
-will not be understood (or retained) with this version.
-</note>
-<note version="8.3" severity="warning">
-Since Version 8.3, EAGLE supports the association of 3D packages
-with devices in libraries, schematics, and board files. Those 3D
-packages will not be understood (or retained) with this version.
-</note>
-</compatibility>
 </eagle>
