File: power-slot/power-slot.brd (EAGLE design)
At the start: 45.8 x 34.3 mm, 9 parts, among them X1 PCB-03-2, X2 PCB-03-2, X3 PCB-03-2

Commit message: Finalize Power slot
Parts:
- removed X3: PCB-03-2, sanisimov:PCB_EDGE_2X3
- added U$5: (no value), microbuilder:SYMBOL_PLUS
- added U$6: (no value), microbuilder:SYMBOL_MINUS
- X1: value PCB-03-2 -> B4B-XH-A; device sanisimov:PCB_EDGE_2X3 -> sanisimov:B4B-XH-A
- X2: value PCB-03-2 -> (none); device sanisimov:PCB_EDGE_2X3 -> sanisimov:FE3-2-CARDEDGE-0.1
- moved C1 37.7 mm to (27.0, 17.5), turned to 0 degrees
- moved X2 36.9 mm to (27.0, 51.0), flipped to the bottom, turned to 90 degrees
- moved U$1 26.6 mm to (19.0, 57.0)
- moved U$2 25.1 mm to (35.0, 57.0)
- moved X1 16.6 mm to (27.0, 10.0), turned to 180 degrees
- moved U$4 16.4 mm to (19.0, 15.0)
- moved PS1 14.8 mm to (27.0, 34.0), turned to 0 degrees
- moved U$3 13.8 mm to (35.0, 15.0)
Connections:
- removed net N$3: X3.2
- removed net PWR: PS1.5, PS1.6, X2.2, X2.3
- new net +5V: PS1.5, PS1.6, X2.4, X2.6
- net GND: now also X1.1, X2.3; no longer X1.2, X1.3, X2.6, X3.3
- net INPWR: now also X1.2; no longer X1.5, X1.6, X3.5, X3.6
- net SCL: now also X1.3, X2.2; no longer X1.4, X2.4, X3.4
- net SDA: now also X1.4; no longer X1.1, X3.1
Routing:
- net SCL: track 0.00 -> 42.3 mm
- net SDA: track 0.00 -> 40.0 mm
- net +5V: track 0.00 -> 21.8 mm
- net INPWR: track 0.00 -> 16.8 mm
- added copper zone on layer 1, net GND
- added copper zone on layer 16, net GND
Other:
- board size 45.8 x 34.3 mm -> 22 x 56 mm
- board text added: "SCL"
- board text added: "SDA"
