File: power-slot/power-slot.sch (EAGLE design)
At the start: 9 parts, among them X1 PCB-03-2, X2 PCB-03-2, X3 PCB-03-2

Commit message: Finalize Power slot
Parts:
- removed X3: PCB-03-2, sanisimov:PCB-03-2
- X1: value PCB-03-2 -> B4B-XH-A; device sanisimov:PCB-03-2 -> sanisimov:B4B-XH-A
- X2: value PCB-03-2 -> (none); device sanisimov:PCB-03-2 -> sanisimov:CON-FE03-2CARDEDGE-0.1
Connections:
- removed net N$3: X3.2
- removed net PWR: PS1.VOUT1+, PS1.VOUT2+, X2.2, X2.3
- new net +5V: PS1.VOUT1+, PS1.VOUT2+, X2.4, X2.6
- net GND: now also X1.1, X2.3; no longer X1.2, X1.3, X2.6, X3.3
- net INPWR: now also X1.2; no longer X1.5, X1.6, X3.5, X3.6
- net SCL: now also X1.3, X2.2; no longer X1.4, X2.4, X3.4
- net SDA: now also X1.4; no longer X1.1, X3.1
Other:
- moved on the sheet: X2
